Commit message: position error minimising in x diredction

File: mecanum/urdf/base.urdf.xacro (robot description, xacro)
@@ -41,5 +41,5 @@
 		<parent link="base_footprint" />
 		<child link="base_link" />
-		<origin xyz="0 0 0.10102" rpy="-1.57079632679 0 0"/>
+		<origin xyz="0 0 0.104" rpy="-1.57079632679 0 0"/>
 	</joint>
     <!-- xyz="0.2 0.054 -0.195" -->
@@ -47,79 +47,79 @@
     name="one"
     color="0.3 0 0"
-    xyz="0.2 0.054 -0.235"
+    xyz="0.2 0.056 -0.236"
     rpy="1.57 0 0"
-    />
+  />
     <!-- xyz="-0.2 0.056 -0.28" -->
-    <xacro:right_rim_macro
+  <xacro:right_rim_macro
     name="two"
     color="0 0.3 0"
     xyz="-0.2 0.056 -0.34"
-      rpy="-1.57 0 0"
-    />
+    rpy="-1.57 0 0"
+  />
     <!-- xyz="-0.2 0.056 0.196" -->
-    <xacro:left_rim_macro
+  <xacro:left_rim_macro
     name="three"
     color="0 0 0.3"
     xyz="-0.2 0.056 0.236"
-      rpy="-1.57 0 0"
-    />
+    rpy="-1.57 0 0"
+  />
     <!-- xyz="0.2 0.056 0.28" -->
-    <xacro:right_rim_macro
+  <xacro:right_rim_macro
     name="four"
     color="0 0 0.3"
     xyz="0.2 0.056 0.34"
-      rpy="1.57 0 0"
-    />
+    rpy="1.57 0 0"
+  />
 	<gazebo reference="base_link">
-    		<material>Gazebo/White</material>
-  	</gazebo>
+  	<material>Gazebo/White</material>
+  </gazebo>
 	<gazebo reference="left_rim_one_link">
-    		<material>Gazebo/Red</material>
-        <mu1>0.2</mu1>
-  		  <mu2>0.2</mu2>
-        <kp>500000.0</kp>
-        <kd>10.0</kd>
-  		  <!-- <selfCollide>true</selfCollide> -->
-  	</gazebo>
+    <material>Gazebo/Red</material>
+    <mu1>0.2</mu1>
+  	<mu2>0.2</mu2>
+    <kp>500000.0</kp>
+    <kd>10.0</kd>
+  	<!-- <selfCollide>true</selfCollide> -->
+  </gazebo>
 	<gazebo reference="right_rim_two_link">
-    		<material>Gazebo/Green</material>
-        <mu1>0.2</mu1>
-  		  <mu2>0.2</mu2>
-        <kp>500000.0</kp>
-        <kd>10.0</kd>
-  		  <!-- <selfCollide>true</selfCollide> -->
-  	</gazebo>
+    <material>Gazebo/Green</material>
+    <mu1>0.2</mu1>
+  	<mu2>0.2</mu2>
+    <kp>500000.0</kp>
+    <kd>10.0</kd>
+  	<!-- <selfCollide>true</selfCollide> -->
+  </gazebo>
 	<gazebo reference="left_rim_three_link">
-    		<material>Gazebo/Blue</material>
-        <mu1>0.2</mu1>
-  		  <mu2>0.2</mu2>
-        <kp>500000.0</kp>
-        <kd>10.0</kd>
-  		  <!-- <selfCollide>true</selfCollide> -->
-  </gazebo>
-    <gazebo reference="right_rim_four_link">
-    		<material>Gazebo/Orange</material>
-        <mu1>0.2</mu1>
-  		  <mu2>0.2</mu2>
-        <kp>500000.0</kp>
-        <kd>10.0</kd>
-  		  <!-- <selfCollide>true</selfCollide> -->
-  	</gazebo>
+    <material>Gazebo/Blue</material>
+    <mu1>0.2</mu1>
+  	<mu2>0.2</mu2>
+    <kp>500000.0</kp>
+    <kd>10.0</kd>
+  	<!-- <selfCollide>true</selfCollide> -->
+  </gazebo>
+  <gazebo reference="right_rim_four_link">
+  	<material>Gazebo/Orange</material>
+    <mu1>0.2</mu1>
+  	<mu2>0.2</mu2>
+    <kp>500000.0</kp>
+    <kd>10.0</kd>
+  	<!-- <selfCollide>true</selfCollide> -->
+  </gazebo>
 	<joint name="imu_joint" type="fixed">
-    	<parent link="base_footprint"/>
-    	<child link="imu_link"/>
-    	<origin xyz="0 0 0.26325" rpy="0 0 0"/>
-  	</joint>
-  	<link name="imu_link"/>
-  	<joint name="scan_joint" type="fixed">
-    	<parent link="base_footprint"/>
-    	<child link="base_scan"/>
-    	<origin xyz="0 0 0.3" rpy="0 0 0"/>
-  	</joint>
-  	<link name="base_scan">
+  	<parent link="base_footprint"/>
+  	<child link="imu_link"/>
+  	<origin xyz="0 0 0.26325" rpy="0 0 0"/>
+  </joint>
+  <link name="imu_link"/>
+  <joint name="scan_joint" type="fixed">
+  	<parent link="base_footprint"/>
+  	<child link="base_scan"/>
+  	<origin xyz="0 0 0.15" rpy="0 0 0"/>
+  </joint>
+  <link name="base_scan">
     <visual>
       <origin xyz="0 0 0.0" rpy="0 0 0"/>
       <geometry>
-        <mesh filename="package://mecanum/meshes/lds.STL" scale="0.001 0.001 0.001"/>
+        <mesh filename="package://mecanum/meshes/lds.stl" scale="0.001 0.001 0.001"/>
       </geometry>
       <material name="dark"/>
@@ -210,5 +210,5 @@
 	  <plugin name="gazebo_ros_control" filename="libgazebo_ros_control.so">
 	    <robotNamespace>/mecanum</robotNamespace>
-      <robotSimType>gazebo_ros_control/DefaultRobotHWSim</robotSimType>
+      <!-- <robotSimType>gazebo_ros_control/DefaultRobotHWSim</robotSimType> -->
 	  </plugin>
 	</gazebo>

File: mecanum/urdf/left_rim.urdf.xacro (robot description, xacro)
@@ -37,4 +37,5 @@
 			<axis xyz="0 1 0"/>
 			<origin xyz="${xyz}" rpy="${rpy}"/>
+      <limit effort="8" velocity="10"/>
 		</joint>
 	 <link
@@ -571,72 +572,72 @@
 	<gazebo reference="${name}_s1">
     <material>Gazebo/Black</material>
-    <mu1>0.5</mu1>
-    <mu2>0.5</mu2>
-    <kp>1000000.0</kp>
-    <kd>100.0</kd>
+    <mu1>1</mu1>
+    <mu2>1</mu2>
+    <kp>10000.0</kp>
+    <kd>1000000.0</kd>
     <!-- <selfCollide>true</selfCollide>  -->
 </gazebo>
 <gazebo reference="${name}_s2">
     <material>Gazebo/Black</material>
-    <mu1>0.5</mu1>
-    <mu2>0.5</mu2>
-    <kp>1000000.0</kp>
-    <kd>100.0</kd>
+    <mu1>1</mu1>
+    <mu2>1</mu2>
+    <kp>10000.0</kp>
+    <kd>1000000.0</kd>
     <!-- <selfCollide>true</selfCollide>  -->
 </gazebo>
 <gazebo reference="${name}_s3">
     <material>Gazebo/Black</material>
-    <mu1>0.5</mu1>
-    <mu2>0.5</mu2>
-    <kp>1000000.0</kp>
-    <kd>100.0</kd>
+    <mu1>1</mu1>
+    <mu2>1</mu2>
+    <kp>10000.0</kp>
+    <kd>1000000.0</kd>
     <!-- <selfCollide>true</selfCollide>  -->
 </gazebo>
 <gazebo reference="${name}_s4">
     <material>Gazebo/Black</material>
-    <mu1>0.5</mu1>
-    <mu2>0.5</mu2>
-    <kp>1000000.0</kp>
-    <kd>100.0</kd>
+    <mu1>1</mu1>
+    <mu2>1</mu2>
+    <kp>10000.0</kp>
+    <kd>1000000.0</kd>
     <!-- <selfCollide>true</selfCollide>  -->
 </gazebo>
 <gazebo reference="${name}_s5">
     <material>Gazebo/Black</material>
-    <mu1>0.5</mu1>
-    <mu2>0.5</mu2>
-    <kp>1000000.0</kp>
-    <kd>100.0</kd>
+    <mu1>1</mu1>
+    <mu2>1</mu2>
+    <kp>10000.0</kp>
+    <kd>1000000.0</kd>
     <!-- <selfCollide>true</selfCollide>  -->
 </gazebo>
 <gazebo reference="${name}_s6">
     <material>Gazebo/Black</material>
-    <mu1>0.5</mu1>
-    <mu2>0.5</mu2>
-    <kp>1000000.0</kp>
-    <kd>100.0</kd>
+    <mu1>1</mu1>
+    <mu2>1</mu2>
+    <kp>10000.0</kp>
+    <kd>1000000.0</kd>
     <!-- <selfCollide>true</selfCollide>  -->
 </gazebo>
 <gazebo reference="${name}_s7">
     <material>Gazebo/Black</material>
-    <mu1>0.5</mu1>
-    <mu2>0.5</mu2>
-    <kp>1000000.0</kp>
-    <kd>100.0</kd>
+    <mu1>1</mu1>
+    <mu2>1</mu2>
+    <kp>10000.0</kp>
+    <kd>1000000.0</kd>
     <!-- <selfCollide>true</selfCollide>  -->
 </gazebo>
 <gazebo reference="${name}_s8">
     <material>Gazebo/Black</material>
-    <mu1>0.5</mu1>
-    <mu2>0.5</mu2>
-    <kp>1000000.0</kp>
-    <kd>100.0</kd>
+    <mu1>1</mu1>
+    <mu2>1</mu2>
+    <kp>10000.0</kp>
+    <kd>1000000.0</kd>
     <!-- <selfCollide>true</selfCollide>  -->
 </gazebo>
 <gazebo reference="${name}_s9">
     <material>Gazebo/Black</material>
-    <mu1>0.5</mu1>
-    <mu2>0.5</mu2>
-    <kp>1000000.0</kp>
-    <kd>100.0</kd>
+    <mu1>1</mu1>
+    <mu2>1</mu2>
+    <kp>10000.0</kp>
+    <kd>1000000.0</kd>
     <!-- <selfCollide>true</selfCollide>  -->
 </gazebo>

File: mecanum/urdf/right_rim.urdf.xacro (robot description, xacro)
@@ -40,4 +40,5 @@
 			<axis xyz="0 1 0"/>
 			<origin xyz="${xyz}" rpy="${rpy}"/>
+      <limit effort="8" velocity="10"/>
 		</joint>
 		<link
@@ -574,72 +575,72 @@
   <gazebo reference="${name}_s2">
     <material>Gazebo/Black</material>
-    <mu1>0.5</mu1>
-    <mu2>0.5</mu2>
-    <kp>1000000.0</kp>
-    <kd>100.0</kd>
+    <mu1>1</mu1>
+    <mu2>1</mu2>
+    <kp>10000.0</kp>
+    <kd>1000000.0</kd>
     <!-- <selfCollide>true</selfCollide> -->
 </gazebo>
 <gazebo reference="${name}_s3">
     <material>Gazebo/Black</material>
-    <mu1>0.5</mu1>
-    <mu2>0.5</mu2>
-    <kp>1000000.0</kp>
-    <kd>100.0</kd>
+    <mu1>1</mu1>
+    <mu2>1</mu2>
+    <kp>10000.0</kp>
+    <kd>1000000.0</kd>
     <!-- <selfCollide>true</selfCollide> -->
 </gazebo>
 <gazebo reference="${name}_s4">
     <material>Gazebo/Black</material>
-    <mu1>0.5</mu1>
-    <mu2>0.5</mu2>
-    <kp>1000000.0</kp>
-    <kd>100.0</kd>
+    <mu1>1</mu1>
+    <mu2>1</mu2>
+    <kp>10000.0</kp>
+    <kd>1000000.0</kd>
     <!-- <selfCollide>true</selfCollide> -->
 </gazebo>
 <gazebo reference="${name}_s5">
     <material>Gazebo/Black</material>
-    <mu1>0.5</mu1>
-    <mu2>0.5</mu2>
-    <kp>1000000.0</kp>
-    <kd>100.0</kd>
+    <mu1>1</mu1>
+    <mu2>1</mu2>
+    <kp>10000.0</kp>
+    <kd>1000000.0</kd>
     <!-- <selfCollide>true</selfCollide> -->
 </gazebo>
 <gazebo reference="${name}_s6">
     <material>Gazebo/Black</material>
-    <mu1>0.5</mu1>
-    <mu2>0.5</mu2>
-    <kp>1000000.0</kp>
-    <kd>100.0</kd>
+    <mu1>1</mu1>
+    <mu2>1</mu2>
+    <kp>10000.0</kp>
+    <kd>1000000.0</kd>
     <!-- <selfCollide>true</selfCollide> -->
 </gazebo>
 <gazebo reference="${name}_s7">
     <material>Gazebo/Black</material>
-    <mu1>0.5</mu1>
-    <mu2>0.5</mu2>
-    <kp>1000000.0</kp>
-    <kd>100.0</kd>
+    <mu1>1</mu1>
+    <mu2>1</mu2>
+    <kp>10000.0</kp>
+    <kd>1000000.0</kd>
     <!-- <selfCollide>true</selfCollide> -->
 </gazebo>
 <gazebo reference="${name}_s8">
     <material>Gazebo/Black</material>
-    <mu1>0.5</mu1>
-    <mu2>0.5</mu2>
-    <kp>1000000.0</kp>
-    <kd>100.0</kd>
+    <mu1>1</mu1>
+    <mu2>1</mu2>
+    <kp>10000.0</kp>
+    <kd>1000000.0</kd>
     <!-- <selfCollide>true</selfCollide> -->
 </gazebo>
 <gazebo reference="${name}_s9">
     <material>Gazebo/Black</material>
-    <mu1>0.5</mu1>
-    <mu2>0.5</mu2>
-    <kp>1000000.0</kp>
-    <kd>100.0</kd>
+    <mu1>1</mu1>
+    <mu2>1</mu2>
+    <kp>10000.0</kp>
+    <kd>1000000.0</kd>
     <!-- <selfCollide>true</selfCollide> -->
 </gazebo>
 <gazebo reference="${name}_s10">
     <material>Gazebo/Black</material>
-    <mu1>0.5</mu1>
-    <mu2>0.5</mu2>
-    <kp>1000000.0</kp>
-    <kd>100.0</kd>
+    <mu1>1</mu1>
+    <mu2>1</mu2>
+    <kp>10000.0</kp>
+    <kd>1000000.0</kd>
     <!-- <selfCollide>true</selfCollide> -->
 </gazebo>
