Commit message: SLAM and Autonomous navigation Donegit status!

File: mecanum/urdf/base.xacro (robot description, xacro)
@@ -1,9 +1,17 @@
 <?xml version="1.0"?>
 <robot xmlns:xacro="http://www.ros.org/wiki/xacro" name="mecanum">
-	<xacro:include filename="$(find mecanum)/urdf/left_rim.urdf.xacro"/>
-  <xacro:include filename="$(find mecanum)/urdf/right_rim.urdf.xacro"/>
+	<xacro:include filename="$(find mecanum)/urdf/left_rim.xacro"/>
+  <xacro:include filename="$(find mecanum)/urdf/right_rim.xacro"/>
+  <xacro:include filename="$(find mecanum)/urdf/encoder_rim.xacro"/>
 	<material name="dark">
     	<color rgba="0.3 0.3 0.3 1.0"/>
   </material>
+	<xacro:arg name="_kp"   default="1e5"/>
+  <xacro:arg name="_kd"   default="1e5"/>
+  <xacro:arg name="_maxVel"   default="40"/>
+  <xacro:arg name="_fdir1_left"   default="1 1 0"/>
+  <xacro:arg name="_fdir1_right"   default="1 -1 0"/>
+  <xacro:arg name="_mu1"   default="10"/>
+  <xacro:arg name="_mu2"   default="10"/>
 	<link name="base_footprint"/>
 	<link name="base_link">
@@ -43,5 +51,4 @@
 		<origin xyz="0 0 0.104" rpy="-1.57079632679 0 0"/>
 	</joint>
-    <!-- xyz="0.2 0.054 -0.195" -->
 	<xacro:left_rim_macro
     name="one"
@@ -50,5 +57,4 @@
     rpy="1.57 0 0"
   />
-    <!-- xyz="-0.2 0.056 -0.28" -->
   <xacro:right_rim_macro
     name="two"
@@ -57,5 +63,4 @@
     rpy="-1.57 0 0"
   />
-    <!-- xyz="-0.2 0.056 0.196" -->
   <xacro:left_rim_macro
     name="three"
@@ -64,5 +69,4 @@
     rpy="-1.57 0 0"
   />
-    <!-- xyz="0.2 0.056 0.28" -->
   <xacro:right_rim_macro
     name="four"
@@ -76,32 +80,32 @@
 	<gazebo reference="left_rim_one_link">
     <material>Gazebo/Red</material>
-    <mu1>0.2</mu1>
-  	<mu2>0.2</mu2>
-    <kp>500000.0</kp>
-    <kd>10.0</kd>
+    <!-- <mu1>0.3</mu1>
+  	<mu2>0.3</mu2>
+    <kp>500000.0</kp>
+    <kd>10.0</kd> -->
   	<!-- <selfCollide>true</selfCollide> -->
   </gazebo>
 	<gazebo reference="right_rim_two_link">
     <material>Gazebo/Green</material>
-    <mu1>0.2</mu1>
-  	<mu2>0.2</mu2>
-    <kp>500000.0</kp>
-    <kd>10.0</kd>
+    <!-- <mu1>0.3</mu1>
+  	<mu2>0.3</mu2>
+    <kp>500000.0</kp>
+    <kd>10.0</kd> -->
   	<!-- <selfCollide>true</selfCollide> -->
   </gazebo>
 	<gazebo reference="left_rim_three_link">
     <material>Gazebo/Blue</material>
-    <mu1>0.2</mu1>
-  	<mu2>0.2</mu2>
-    <kp>500000.0</kp>
-    <kd>10.0</kd>
+    <!-- <mu1>0.3</mu1>
+  	<mu2>0.3</mu2>
+    <kp>500000.0</kp>
+    <kd>10.0</kd> -->
   	<!-- <selfCollide>true</selfCollide> -->
   </gazebo>
   <gazebo reference="right_rim_four_link">
   	<material>Gazebo/Orange</material>
-    <mu1>0.2</mu1>
-  	<mu2>0.2</mu2>
-    <kp>500000.0</kp>
-    <kd>10.0</kd>
+    <!-- <mu1>0.3</mu1>
+  	<mu2>0.3</mu2>
+    <kp>500000.0</kp>
+    <kd>10.0</kd> -->
   	<!-- <selfCollide>true</selfCollide> -->
   </gazebo>
@@ -192,5 +196,5 @@
         <range>
           <min>0.120</min>
-          <max>3.5</max>
+          <max>10</max>
           <resolution>0.015</resolution>
         </range>
@@ -207,4 +211,38 @@
     </sensor>
   </gazebo>
+  <!-- holonomic encoder setup -->
+  <xacro:encoder_macro
+    name="one"
+    color="0.3 0 0"
+    xyz="0.04 0.08 0"
+    rpy="0 -1.570796327 0"/>
+  <xacro:encoder_macro
+    name="two"
+    color="0 0.3 0"
+    xyz="-0.02 0.08 0.034641016"
+    rpy="0 2.617993878 0"/>
+  <xacro:encoder_macro
+    name="three"
+    color="0 0 0.3"
+    xyz="-0.02 0.08 -0.03464101615"
+    rpy="0 0.523598776 0"/>
+  <gazebo reference="encoder_one_link">
+  	<material>Gazebo/Red</material>
+    <mu1>$(arg _mu1)</mu1>
+  	<mu2>$(arg _mu2)</mu2>
+  	<selfCollide>true</selfCollide>
+  </gazebo>
+	<gazebo reference="encoder_two_link">
+  	<material>Gazebo/Green</material>
+    <mu1>$(arg _mu1)</mu1>
+  	<mu2>$(arg _mu2)</mu2>
+  	<selfCollide>true</selfCollide>
+  </gazebo>
+	<gazebo reference="encoder_three_link">
+  	<material>Gazebo/Blue</material>
+    <mu1>$(arg _mu1)</mu1>
+  	<mu2>$(arg _mu2)</mu2>
+  	<selfCollide>true</selfCollide>
+  </gazebo>
   <gazebo>
 	  <plugin name="gazebo_ros_control" filename="libgazebo_ros_control.so">

File: mecanum/urdf/left_rim.xacro (robot description, xacro)
@@ -37,5 +37,5 @@
 			<axis xyz="0 1 0"/>
 			<origin xyz="${xyz}" rpy="${rpy}"/>
-      <limit effort="8" velocity="10"/>
+      <limit effort="8" velocity="$(arg _maxVel)"/>
 		</joint>
 	 <link
@@ -91,10 +91,7 @@
     <axis
       xyz="0 1 0" />
-    <!-- <limit
-      effort="100"
-      velocity="100" />
-    <dynamics
-      damping="0.1"
-      friction="0.1" /> -->
+    <limit
+      effort="0"
+      velocity="$(arg _maxVel)" />
   </joint>
   <link
@@ -150,10 +147,7 @@
     <axis
       xyz="0 1 0" />
-    <!-- <limit
-      effort="100"
-      velocity="100" />
-    <dynamics
-      damping="0.1"
-      friction="0.1" /> -->
+    <limit
+      effort="0"
+      velocity="$(arg _maxVel)" />
   </joint>
   <link
@@ -209,10 +203,7 @@
     <axis
       xyz="0 1 0" />
-    <!-- <limit
-      effort="100"
-      velocity="100" />
-    <dynamics
-      damping="0.1"
-      friction="0.1" /> -->
+    <limit
+      effort="0"
+      velocity="$(arg _maxVel)" />
   </joint>
   <link
@@ -268,10 +259,7 @@
     <axis
       xyz="0 1 0" />
-    <!-- <limit
-      effort="100"
-      velocity="100" />
-    <dynamics
-      damping="0.1"
-      friction="0.1" /> -->
+    <limit
+      effort="0"
+      velocity="$(arg _maxVel)" />
   </joint>
   <link
@@ -327,10 +315,7 @@
     <axis
       xyz="0 1 0" />
-    <!-- <limit
-      effort="100"
-      velocity="100" />
-    <dynamics
-      damping="0.1"
-      friction="0.1" /> -->
+    <limit
+      effort="0"
+      velocity="$(arg _maxVel)" />
   </joint>
   <link
@@ -386,10 +371,7 @@
     <axis
       xyz="0 1 0" />
-    <!-- <limit
-      effort="100"
-      velocity="100" />
-    <dynamics
-      damping="0.1"
-      friction="0.1" /> -->
+    <limit
+      effort="0"
+      velocity="$(arg _maxVel)" />
   </joint>
   <link
@@ -445,10 +427,7 @@
     <axis
       xyz="0 1 0" />
-    <!-- <limit
-      effort="100"
-      velocity="100" />
-    <dynamics
-      damping="0.1"
-      friction="0.1" /> -->
+    <limit
+      effort="0"
+      velocity="$(arg _maxVel)" />
   </joint>
   <link
@@ -504,10 +483,7 @@
     <axis
       xyz="0 1 0" />
-    <!-- <limit
-      effort="100"
-      velocity="100" />
-    <dynamics
-      damping="0.1"
-      friction="0.1" /> -->
+    <limit
+      effort="0"
+      velocity="$(arg _maxVel)" />
   </joint>
   <link
@@ -563,81 +539,105 @@
     <axis
       xyz="0 1 0" />
-    <!-- <limit
-      effort="100"
-      velocity="100" />
-    <dynamics
-      damping="0.1"
-      friction="0.1" /> -->
+    <limit
+      effort="0"
+      velocity="$(arg _maxVel)" />
   </joint>
 	<gazebo reference="${name}_s1">
     <material>Gazebo/Black</material>
-    <mu1>1</mu1>
-    <mu2>1</mu2>
-    <kp>10000.0</kp>
-    <kd>1000000.0</kd>
+    <mu1>$(arg _mu1)</mu1>
+    <mu2>$(arg _mu2)</mu2>
+    <kp>$(arg _kp)</kp>
+    <kd>$(arg _kd)</kd>
+    <minDepth>0.001</minDepth>
+    <maxVel>$(arg _maxVel)</maxVel>
+    <fdir1>$(arg _fdir1_left)</fdir1>
     <!-- <selfCollide>true</selfCollide>  -->
 </gazebo>
 <gazebo reference="${name}_s2">
     <material>Gazebo/Black</material>
-    <mu1>1</mu1>
-    <mu2>1</mu2>
-    <kp>10000.0</kp>
-    <kd>1000000.0</kd>
+    <mu1>$(arg _mu1)</mu1>
+    <mu2>$(arg _mu2)</mu2>
+    <kp>$(arg _kp)</kp>
+    <kd>$(arg _kd)</kd>
+    <minDepth>0.001</minDepth>
+    <maxVel>$(arg _maxVel)</maxVel>
+    <fdir1>$(arg _fdir1_left)</fdir1>
     <!-- <selfCollide>true</selfCollide>  -->
 </gazebo>
 <gazebo reference="${name}_s3">
     <material>Gazebo/Black</material>
-    <mu1>1</mu1>
-    <mu2>1</mu2>
-    <kp>10000.0</kp>
-    <kd>1000000.0</kd>
+    <mu1>$(arg _mu1)</mu1>
+    <mu2>$(arg _mu2)</mu2>
+    <kp>$(arg _kp)</kp>
+    <kd>$(arg _kd)</kd>
+    <minDepth>0.001</minDepth>
+    <maxVel>$(arg _maxVel)</maxVel>
+    <fdir1>$(arg _fdir1_left)</fdir1>
     <!-- <selfCollide>true</selfCollide>  -->
 </gazebo>
 <gazebo reference="${name}_s4">
     <material>Gazebo/Black</material>
-    <mu1>1</mu1>
-    <mu2>1</mu2>
-    <kp>10000.0</kp>
-    <kd>1000000.0</kd>
+    <mu1>$(arg _mu1)</mu1>
+    <mu2>$(arg _mu2)</mu2>
+    <kp>$(arg _kp)</kp>
+    <kd>$(arg _kd)</kd>
+    <minDepth>0.001</minDepth>
+    <maxVel>$(arg _maxVel)</maxVel>
+    <fdir1>$(arg _fdir1_left)</fdir1>
     <!-- <selfCollide>true</selfCollide>  -->
 </gazebo>
 <gazebo reference="${name}_s5">
     <material>Gazebo/Black</material>
-    <mu1>1</mu1>
-    <mu2>1</mu2>
-    <kp>10000.0</kp>
-    <kd>1000000.0</kd>
+    <mu1>$(arg _mu1)</mu1>
+    <mu2>$(arg _mu2)</mu2>
+    <kp>$(arg _kp)</kp>
+    <kd>$(arg _kd)</kd>
+    <minDepth>0.001</minDepth>
+    <maxVel>$(arg _maxVel)</maxVel>
+    <fdir1>$(arg _fdir1_left)</fdir1>
     <!-- <selfCollide>true</selfCollide>  -->
 </gazebo>
 <gazebo reference="${name}_s6">
     <material>Gazebo/Black</material>
-    <mu1>1</mu1>
-    <mu2>1</mu2>
-    <kp>10000.0</kp>
-    <kd>1000000.0</kd>
+    <mu1>$(arg _mu1)</mu1>
+    <mu2>$(arg _mu2)</mu2>
+    <kp>$(arg _kp)</kp>
+    <kd>$(arg _kd)</kd>
+    <minDepth>0.001</minDepth>
+    <maxVel>$(arg _maxVel)</maxVel>
+    <fdir1>$(arg _fdir1_left)</fdir1>
     <!-- <selfCollide>true</selfCollide>  -->
 </gazebo>
 <gazebo reference="${name}_s7">
     <material>Gazebo/Black</material>
-    <mu1>1</mu1>
-    <mu2>1</mu2>
-    <kp>10000.0</kp>
-    <kd>1000000.0</kd>
+    <mu1>$(arg _mu1)</mu1>
+    <mu2>$(arg _mu2)</mu2>
+    <kp>$(arg _kp)</kp>
+    <kd>$(arg _kd)</kd>
+    <minDepth>0.001</minDepth>
+    <maxVel>$(arg _maxVel)</maxVel>
+    <fdir1>$(arg _fdir1_left)</fdir1>
     <!-- <selfCollide>true</selfCollide>  -->
 </gazebo>
 <gazebo reference="${name}_s8">
     <material>Gazebo/Black</material>
-    <mu1>1</mu1>
-    <mu2>1</mu2>
-    <kp>10000.0</kp>
-    <kd>1000000.0</kd>
+    <mu1>$(arg _mu1)</mu1>
+    <mu2>$(arg _mu2)</mu2>
+    <kp>$(arg _kp)</kp>
+    <kd>$(arg _kd)</kd>
+    <minDepth>0.001</minDepth>
+    <maxVel>$(arg _maxVel)</maxVel>
+    <fdir1>$(arg _fdir1_left)</fdir1>
     <!-- <selfCollide>true</selfCollide>  -->
 </gazebo>
 <gazebo reference="${name}_s9">
     <material>Gazebo/Black</material>
-    <mu1>1</mu1>
-    <mu2>1</mu2>
-    <kp>10000.0</kp>
-    <kd>1000000.0</kd>
+    <mu1>$(arg _mu1)</mu1>
+    <mu2>$(arg _mu2)</mu2>
+    <kp>$(arg _kp)</kp>
+    <kd>$(arg _kd)</kd>
+    <minDepth>0.001</minDepth>
+    <maxVel>$(arg _maxVel)</maxVel>
+    <fdir1>$(arg _fdir1_left)</fdir1>
     <!-- <selfCollide>true</selfCollide>  -->
 </gazebo>

File: mecanum/urdf/right_rim.xacro (robot description, xacro)
@@ -40,5 +40,5 @@
 			<axis xyz="0 1 0"/>
 			<origin xyz="${xyz}" rpy="${rpy}"/>
-      <limit effort="8" velocity="10"/>
+      <limit effort="8" velocity="$(arg _maxVel)"/>
 		</joint>
 		<link
@@ -94,10 +94,7 @@
     <axis
       xyz="0 1 0" />
-    <!-- <limit
-      effort="100"
-      velocity="100" />
-    <dynamics
-      damping="0.1"
-      friction="0.1" /> -->
+    <limit
+      effort="0"
+      velocity="$(arg _maxVel)" />
   </joint>
   <link
@@ -153,10 +150,7 @@
     <axis
       xyz="0 1 0" />
-    <!-- <limit
-      effort="100"
-      velocity="100" />
-    <dynamics
-      damping="0.1"
-      friction="0.1" /> -->
+    <limit
+      effort="0"
+      velocity="$(arg _maxVel)" />
   </joint>
   <link
@@ -212,10 +206,7 @@
     <axis
       xyz="0 1 0" />
-    <!-- <limit
-      effort="100"
-      velocity="100" />
-    <dynamics
-      damping="0.1"
-      friction="0.1" /> -->
+    <limit
+      effort="0"
+      velocity="$(arg _maxVel)" />
   </joint>
   <link
@@ -271,10 +262,7 @@
     <axis
       xyz="0 1 0" />
-    <!-- <limit
-      effort="100"
-      velocity="100" />
-    <dynamics
-      damping="0.1"
-      friction="0.1" /> -->
+    <limit
+      effort="0"
+      velocity="$(arg _maxVel)" />
   </joint>
   <link
@@ -330,10 +318,7 @@
     <axis
       xyz="0 1 0" />
-    <!-- <limit
-      effort="100"
-      velocity="100" />
-    <dynamics
-      damping="0.1"
-      friction="0.1" /> -->
+    <limit
+      effort="0"
+      velocity="$(arg _maxVel)" />
   </joint>
   <link
@@ -389,10 +374,7 @@
     <axis
       xyz="0 1 0" />
-    <!-- <limit
-      effort="100"
-      velocity="100" />
-    <dynamics
-      damping="0.1"
-      friction="0.1" /> -->
+    <limit
+      effort="0"
+      velocity="$(arg _maxVel)" />
   </joint>
   <link
@@ -448,10 +430,7 @@
     <axis
       xyz="0 1 0" />
-    <!-- <limit
-      effort="100"
-      velocity="100" />
-    <dynamics
-      damping="0.1"
-      friction="0.1" /> -->
+    <limit
+      effort="0"
+      velocity="$(arg _maxVel)" />
   </joint>
   <link
@@ -507,10 +486,7 @@
     <axis
       xyz="0 1 0" />
-    <!-- <limit
-      effort="100"
-      velocity="100" />
-    <dynamics
-      damping="0.1"
-      friction="0.1" /> -->
+    <limit
+      effort="0"
+      velocity="$(arg _maxVel)" />
   </joint>
   <link
@@ -566,81 +542,105 @@
     <axis
       xyz="0 -1 0" />
-    <!-- <limit
-      effort="100"
-      velocity="100" />
-    <dynamics
-      damping="0.1"
-      friction="0.1" /> -->
+    <limit
+      effort="0"
+      velocity="$(arg _maxVel)" />
   </joint>
   <gazebo reference="${name}_s2">
     <material>Gazebo/Black</material>
-    <mu1>1</mu1>
-    <mu2>1</mu2>
-    <kp>10000.0</kp>
-    <kd>1000000.0</kd>
+    <mu1>$(arg _mu1)</mu1>
+    <mu2>$(arg _mu2)</mu2>
+    <kp>$(arg _kp)</kp>
+    <kp>$(arg _kd)</kp>
+    <minDepth>0.001</minDepth>
+    <maxVel>$(arg _maxVel)</maxVel>
+    <fdir1>$(arg _fdir1_right)</fdir1>
     <!-- <selfCollide>true</selfCollide> -->
 </gazebo>
 <gazebo reference="${name}_s3">
     <material>Gazebo/Black</material>
-    <mu1>1</mu1>
-    <mu2>1</mu2>
-    <kp>10000.0</kp>
-    <kd>1000000.0</kd>
+    <mu1>$(arg _mu1)</mu1>
+    <mu2>$(arg _mu2)</mu2>
+    <kp>$(arg _kp)</kp>
+    <kp>$(arg _kd)</kp>
+    <minDepth>0.001</minDepth>
+    <maxVel>$(arg _maxVel)</maxVel>
+    <fdir1>$(arg _fdir1_right)</fdir1>
     <!-- <selfCollide>true</selfCollide> -->
 </gazebo>
 <gazebo reference="${name}_s4">
     <material>Gazebo/Black</material>
-    <mu1>1</mu1>
-    <mu2>1</mu2>
-    <kp>10000.0</kp>
-    <kd>1000000.0</kd>
+    <mu1>$(arg _mu1)</mu1>
+    <mu2>$(arg _mu2)</mu2>
+    <kp>$(arg _kp)</kp>
+    <kp>$(arg _kd)</kp>
+    <minDepth>0.001</minDepth>
+    <maxVel>$(arg _maxVel)</maxVel>
+    <fdir1>$(arg _fdir1_right)</fdir1>
     <!-- <selfCollide>true</selfCollide> -->
 </gazebo>
 <gazebo reference="${name}_s5">
     <material>Gazebo/Black</material>
-    <mu1>1</mu1>
-    <mu2>1</mu2>
-    <kp>10000.0</kp>
-    <kd>1000000.0</kd>
+    <mu1>$(arg _mu1)</mu1>
+    <mu2>$(arg _mu2)</mu2>
+    <kp>$(arg _kp)</kp>
+    <kp>$(arg _kd)</kp>
+    <minDepth>0.001</minDepth>
+    <maxVel>$(arg _maxVel)</maxVel>
+    <fdir1>$(arg _fdir1_right)</fdir1>
     <!-- <selfCollide>true</selfCollide> -->
 </gazebo>
 <gazebo reference="${name}_s6">
     <material>Gazebo/Black</material>
-    <mu1>1</mu1>
-    <mu2>1</mu2>
-    <kp>10000.0</kp>
-    <kd>1000000.0</kd>
+    <mu1>$(arg _mu1)</mu1>
+    <mu2>$(arg _mu2)</mu2>
+    <kp>$(arg _kp)</kp>
+    <kp>$(arg _kd)</kp>
+    <minDepth>0.001</minDepth>
+    <maxVel>$(arg _maxVel)</maxVel>
+    <fdir1>$(arg _fdir1_right)</fdir1>
     <!-- <selfCollide>true</selfCollide> -->
 </gazebo>
 <gazebo reference="${name}_s7">
     <material>Gazebo/Black</material>
-    <mu1>1</mu1>
-    <mu2>1</mu2>
-    <kp>10000.0</kp>
-    <kd>1000000.0</kd>
+    <mu1>$(arg _mu1)</mu1>
+    <mu2>$(arg _mu2)</mu2>
+    <kp>$(arg _kp)</kp>
+    <kp>$(arg _kd)</kp>
+    <minDepth>0.001</minDepth>
+    <maxVel>$(arg _maxVel)</maxVel>
+    <fdir1>$(arg _fdir1_right)</fdir1>
     <!-- <selfCollide>true</selfCollide> -->
 </gazebo>
 <gazebo reference="${name}_s8">
     <material>Gazebo/Black</material>
-    <mu1>1</mu1>
-    <mu2>1</mu2>
-    <kp>10000.0</kp>
-    <kd>1000000.0</kd>
+    <mu1>$(arg _mu1)</mu1>
+    <mu2>$(arg _mu2)</mu2>
+    <kp>$(arg _kp)</kp>
+    <kp>$(arg _kd)</kp>
+    <minDepth>0.001</minDepth>
+    <maxVel>$(arg _maxVel)</maxVel>
+    <fdir1>$(arg _fdir1_right)</fdir1>
     <!-- <selfCollide>true</selfCollide> -->
 </gazebo>
 <gazebo reference="${name}_s9">
     <material>Gazebo/Black</material>
-    <mu1>1</mu1>
-    <mu2>1</mu2>
-    <kp>10000.0</kp>
-    <kd>1000000.0</kd>
+    <mu1>$(arg _mu1)</mu1>
+    <mu2>$(arg _mu2)</mu2>
+    <kp>$(arg _kp)</kp>
+    <kp>$(arg _kd)</kp>
+    <minDepth>0.001</minDepth>
+    <maxVel>$(arg _maxVel)</maxVel>
+    <fdir1>$(arg _fdir1_right)</fdir1>
     <!-- <selfCollide>true</selfCollide> -->
 </gazebo>
 <gazebo reference="${name}_s10">
     <material>Gazebo/Black</material>
-    <mu1>1</mu1>
-    <mu2>1</mu2>
-    <kp>10000.0</kp>
-    <kd>1000000.0</kd>
+    <mu1>$(arg _mu1)</mu1>
+    <mu2>$(arg _mu2)</mu2>
+    <kp>$(arg _kp)</kp>
+    <kp>$(arg _kd)</kp>
+    <minDepth>0.001</minDepth>
+    <maxVel>$(arg _maxVel)</maxVel>
+    <fdir1>$(arg _fdir1_right)</fdir1>
     <!-- <selfCollide>true</selfCollide> -->
 </gazebo>
